Commit message: For Experiments

File: limo_ros2/limo_description/urdf/limo_four_diff.xacro (robot description, xacro)
@@ -2,4 +2,6 @@
 <robot name="limo_four_diff" xmlns:xacro="http://ros.org/wiki/xacro">
     <xacro:include filename="$(find limo_description)/urdf/limo_xacro.xacro" />
+    <xacro:arg name="tf_prefix" default="" />
+    <xacro:property name="tf_prefix" value="$(arg tf_prefix)" />
     <!-- Variables -->
     <xacro:property name="M_PI" value="3.14159"/>
@@ -15,5 +17,5 @@
     <xacro:property name="wheel_radius" value="0.045" />
     <!-- Base link -->
-    <link name="base_link">
+    <link name="${tf_prefix}base_link">
         <visual>
             <origin xyz="0 0 -0.15" rpy="0 0 1.57" />
@@ -30,5 +32,5 @@
         </collision>
     </link>
-    <link name="inertial_link">
+    <link name="${tf_prefix}inertial_link">
         <inertial>
             <origin xyz="0.0 0.0 0.0" />
@@ -39,25 +41,25 @@
         </inertial>
     </link>
-    <joint name="inertial_joint" type="fixed">
+    <joint name="${tf_prefix}inertial_joint" type="fixed">
         <origin xyz="0 0 0" rpy="0 0 0" />
-        <parent link="base_link" />
-        <child link="inertial_link" />
+        <parent link="${tf_prefix}base_link" />
+        <child link="${tf_prefix}inertial_link" />
     </joint>
-    <xacro:limo_laser parent_prefix="base_link" frame_prefix="laser">
+    <xacro:limo_laser parent_prefix="${tf_prefix}base_link" frame_prefix="${tf_prefix}laser">
         <origin xyz="0.103 0 -0.034" rpy="0 0 0"/>
     </xacro:limo_laser>
-    <xacro:limo_imu parent_prefix="base_link" frame_prefix="imu">
+    <xacro:limo_imu parent_prefix="${tf_prefix}base_link" frame_prefix="${tf_prefix}imu">
         <origin xyz="0.0 0 -0.1" rpy="0 0 0"/>
     </xacro:limo_imu>
-    <xacro:limo_wheel parent_prefix="base_link" wheel_prefix="front_left" reflect="1">
+    <xacro:limo_wheel parent_prefix="${tf_prefix}base_link" wheel_prefix="${tf_prefix}front_left" reflect="1">
         <origin xyz="${wheelbase/2} ${track/2} ${wheel_vertical_offset}" rpy="0 0  0" />
     </xacro:limo_wheel>
-    <xacro:limo_wheel parent_prefix="base_link" wheel_prefix="front_right" reflect="-1">
+    <xacro:limo_wheel parent_prefix="${tf_prefix}base_link" wheel_prefix="${tf_prefix}front_right" reflect="-1">
         <origin xyz="${wheelbase/2} ${-track/2} ${wheel_vertical_offset}" rpy="${M_PI} 0 0" />
     </xacro:limo_wheel>
-    <xacro:limo_wheel parent_prefix="base_link" wheel_prefix="rear_left" reflect="1">
+    <xacro:limo_wheel parent_prefix="${tf_prefix}base_link" wheel_prefix="${tf_prefix}rear_left" reflect="1">
         <origin xyz="${-wheelbase/2} ${track/2} ${wheel_vertical_offset}" rpy="0 0 0" />
     </xacro:limo_wheel>
-    <xacro:limo_wheel parent_prefix="base_link" wheel_prefix="rear_right" reflect="-1">
+    <xacro:limo_wheel parent_prefix="${tf_prefix}base_link" wheel_prefix="${tf_prefix}rear_right" reflect="-1">
         <origin xyz="${-wheelbase/2} ${-track/2} ${wheel_vertical_offset}" rpy="${M_PI} 0 0" />
     </xacro:limo_wheel>

File: limo_ros2/limo_description/urdf/limo_xacro.xacro (robot description, xacro)
@@ -59,5 +59,5 @@
             </collision>
         </link>
-        <joint type="fixed" name="laser_joint">
+        <joint type="fixed" name="${frame_prefix}_joint">
             <xacro:insert_block name="joint_pose"/>
             <child link="${frame_prefix}_link"/>
@@ -99,5 +99,5 @@
             </collision>
         </link>
-        <joint type="fixed" name="imu_joint">
+        <joint type="fixed" name="${frame_prefix}_joint">
             <xacro:insert_block name="joint_pose"/>
             <child link="${frame_prefix}_link"/>
